File: pcb/chocofi.kicad_pcb (KiCad board)
At the start: 2 copper layers, 111.3 x 90 mm, 60 parts, among them J1 MJ-4PP-9, J2 OLED, J3 Conn_01x02_Female, SW1 SW_SPDT, SW10 SW_PUSH, SW11 SW_PUSH, SW12 SW_PUSH, SW14 SW_PUSH, SW15 SW_PUSH, SW16 SW_PUSH, SW17 SW_PUSH, SW18 SW_PUSH, SW19 SW_PUSH, SW2 SW_PUSH, SW2 SW_SPDT, SW20 SW_PUSH, SW21 SW_PUSH, SW3 SW_PUSH, SW4 SW_PUSH, SW5 SW_PUSH, SW6 SW_PUSH, SW8 SW_PUSH, SW9 SW_PUSH, U1 ProMicro

Commit message: feat: update
Parts:
- added C1: 100nF, Capacitor_SMD:C_0805_2012Metric_Pad1.18x1.45mm_HandSolder, F.Cu at (385.8, 122.1)
- added C10: 100nF, Capacitor_SMD:C_0805_2012Metric_Pad1.18x1.45mm_HandSolder, F.Cu at (390.6, 125.1)
- added C11: 100nF, Capacitor_SMD:C_0805_2012Metric_Pad1.18x1.45mm_HandSolder, F.Cu at (390.6, 128.1)
- added C12: 100nF, Capacitor_SMD:C_0805_2012Metric_Pad1.18x1.45mm_HandSolder, F.Cu at (390.6, 131.1)
- added C13: 100nF, Capacitor_SMD:C_0805_2012Metric_Pad1.18x1.45mm_HandSolder, F.Cu at (390.6, 134.1)
- added C14: 100nF, Capacitor_SMD:C_0805_2012Metric_Pad1.18x1.45mm_HandSolder, F.Cu at (390.6, 137.1)
- added C15: 100nF, Capacitor_SMD:C_0805_2012Metric_Pad1.18x1.45mm_HandSolder, F.Cu at (390.6, 140.1)
- added C16: 100nF, Capacitor_SMD:C_0805_2012Metric_Pad1.18x1.45mm_HandSolder, F.Cu at (390.6, 143.1)
- added C17: 100nF, Capacitor_SMD:C_0805_2012Metric_Pad1.18x1.45mm_HandSolder, F.Cu at (395.4, 122.1)
- added C18: 100nF, Capacitor_SMD:C_0805_2012Metric_Pad1.18x1.45mm_HandSolder, F.Cu at (395.4, 125.1)
- added C19: 100nF, Capacitor_SMD:C_0805_2012Metric_Pad1.18x1.45mm_HandSolder, F.Cu at (395.4, 128.1)
- added C2: 100nF, Capacitor_SMD:C_0805_2012Metric_Pad1.18x1.45mm_HandSolder, F.Cu at (385.8, 125.1)
- added C20: 100nF, Capacitor_SMD:C_0805_2012Metric_Pad1.18x1.45mm_HandSolder, F.Cu at (395.4, 131.1)
- added C21: 100nF, Capacitor_SMD:C_0805_2012Metric_Pad1.18x1.45mm_HandSolder, F.Cu at (395.4, 134.1)
- added C22: 100nF, Capacitor_SMD:C_0805_2012Metric_Pad1.18x1.45mm_HandSolder, F.Cu at (395.4, 137.1)
- added C23: 100nF, Capacitor_SMD:C_0805_2012Metric_Pad1.18x1.45mm_HandSolder, F.Cu at (395.4, 140.1)
- added C24: 100nF, Capacitor_SMD:C_0805_2012Metric_Pad1.18x1.45mm_HandSolder, F.Cu at (395.4, 143.1)
- added C25: 100nF, Capacitor_SMD:C_0805_2012Metric_Pad1.18x1.45mm_HandSolder, F.Cu at (400.2, 122.1)
- added C26: 100nF, Capacitor_SMD:C_0805_2012Metric_Pad1.18x1.45mm_HandSolder, F.Cu at (400.2, 125.1)
- added C27: 100nF, Capacitor_SMD:C_0805_2012Metric_Pad1.18x1.45mm_HandSolder, F.Cu at (400.2, 128.1)
- added C28: 100nF, Capacitor_SMD:C_0805_2012Metric_Pad1.18x1.45mm_HandSolder, F.Cu at (400.2, 131.1)
- added C29: 100nF, Capacitor_SMD:C_0805_2012Metric_Pad1.18x1.45mm_HandSolder, F.Cu at (400.2, 134.1)
- added C3: 100nF, Capacitor_SMD:C_0805_2012Metric_Pad1.18x1.45mm_HandSolder, F.Cu at (385.8, 128.1)
- added C30: 100nF, Capacitor_SMD:C_0805_2012Metric_Pad1.18x1.45mm_HandSolder, F.Cu at (400.2, 137.1)
- added C31: 100nF, Capacitor_SMD:C_0805_2012Metric_Pad1.18x1.45mm_HandSolder, F.Cu at (400.2, 140.1)
- added C32: 100nF, Capacitor_SMD:C_0805_2012Metric_Pad1.18x1.45mm_HandSolder, F.Cu at (400.2, 143.1)
- added C33: 100nF, Capacitor_SMD:C_0805_2012Metric_Pad1.18x1.45mm_HandSolder, F.Cu at (405.0, 122.1)
- added C34: 100nF, Capacitor_SMD:C_0805_2012Metric_Pad1.18x1.45mm_HandSolder, F.Cu at (405.0, 125.1)
- added C35: 100nF, Capacitor_SMD:C_0805_2012Metric_Pad1.18x1.45mm_HandSolder, F.Cu at (405.0, 128.1)
- added C36: 100nF, Capacitor_SMD:C_0805_2012Metric_Pad1.18x1.45mm_HandSolder, F.Cu at (405.0, 131.1)
- added C4: 100nF, Capacitor_SMD:C_0805_2012Metric_Pad1.18x1.45mm_HandSolder, F.Cu at (385.8, 131.1)
- added C5: 100nF, Capacitor_SMD:C_0805_2012Metric_Pad1.18x1.45mm_HandSolder, F.Cu at (385.8, 134.1)
- added C6: 100nF, Capacitor_SMD:C_0805_2012Metric_Pad1.18x1.45mm_HandSolder, F.Cu at (385.8, 137.1)
- added C7: 100nF, Capacitor_SMD:C_0805_2012Metric_Pad1.18x1.45mm_HandSolder, F.Cu at (385.8, 140.1)
- added C8: 100nF, Capacitor_SMD:C_0805_2012Metric_Pad1.18x1.45mm_HandSolder, F.Cu at (385.8, 143.1)
- added C9: 100nF, Capacitor_SMD:C_0805_2012Metric_Pad1.18x1.45mm_HandSolder, F.Cu at (390.6, 122.1)
- added Cap100nf1: C, Capacitor_SMD:C_0805_2012Metric_Pad1.18x1.45mm_HandSolder, F.Cu at (405.0, 134.1)
- added Cap100nf2: C, Capacitor_SMD:C_0805_2012Metric_Pad1.18x1.45mm_HandSolder, F.Cu at (405.0, 137.1)
- added D1: SK6812MINI, LED_SMD:LED_SK6812MINI_PLCC4_3.5x3.5mm_P1.75mm, F.Cu at (386.7, 54.1)
- added D13: SK6812MINI, LED_SMD:LED_SK6812MINI_PLCC4_3.5x3.5mm_P1.75mm, F.Cu at (386.7, 64.3)
- added D22: SK6812MINI, LED_SMD:LED_SK6812MINI_PLCC4_3.5x3.5mm_P1.75mm, F.Cu at (386.7, 69.4)
- added D23: D, Diode_SMD:D_SOD-323_HandSoldering, F.Cu at (410.0, 122.0)
- added D24: D, Diode_SMD:D_SOD-323_HandSoldering, F.Cu at (410.0, 125.0)
- added D25: D, Diode_SMD:D_SOD-323_HandSoldering, F.Cu at (410.0, 127.9)
- added D26: D, Diode_SMD:D_SOD-323_HandSoldering, F.Cu at (410.0, 130.9)
- added D27: D, Diode_SMD:D_SOD-323_HandSoldering, F.Cu at (410.0, 133.8)
- added D28: SK6812MINI, LED_SMD:LED_SK6812MINI_PLCC4_3.5x3.5mm_P1.75mm, F.Cu at (386.7, 74.6)
- added D29: D, Diode_SMD:D_SOD-323_HandSoldering, F.Cu at (410.0, 136.8)
- added D30: D, Diode_SMD:D_SOD-323_HandSoldering, F.Cu at (410.0, 139.7)
- added D31: D, Diode_SMD:D_SOD-323_HandSoldering, F.Cu at (415.1, 122.0)
- added D32: D, Diode_SMD:D_SOD-323_HandSoldering, F.Cu at (415.1, 125.0)
- added D33: D, Diode_SMD:D_SOD-323_HandSoldering, F.Cu at (415.1, 127.9)
- added D34: SK6812MINI, LED_SMD:LED_SK6812MINI_PLCC4_3.5x3.5mm_P1.75mm, F.Cu at (386.7, 79.7)
- added D35: D, Diode_SMD:D_SOD-323_HandSoldering, F.Cu at (415.1, 130.9)
- added D36: D, Diode_SMD:D_SOD-323_HandSoldering, F.Cu at (415.1, 133.8)
- added D37: D, Diode_SMD:D_SOD-323_HandSoldering, F.Cu at (415.1, 136.8)
- added D38: D, Diode_SMD:D_SOD-323_HandSoldering, F.Cu at (415.1, 139.7)
- added D39: D, Diode_SMD:D_SOD-323_HandSoldering, F.Cu at (420.2, 122.0)
- added D40: D, Diode_SMD:D_SOD-323_HandSoldering, F.Cu at (420.2, 125.0)
- added D41: D, Diode_SMD:D_SOD-323_HandSoldering, F.Cu at (420.2, 127.9)
- added D42: D, Diode_SMD:D_SOD-323_HandSoldering, F.Cu at (420.2, 130.9)
- added D43: SK6812MINI, LED_SMD:LED_SK6812MINI_PLCC4_3.5x3.5mm_P1.75mm, F.Cu at (393.4, 54.1)
- added D44: SK6812MINI, LED_SMD:LED_SK6812MINI_PLCC4_3.5x3.5mm_P1.75mm, F.Cu at (393.4, 59.2)
- added D45: SK6812MINI, LED_SMD:LED_SK6812MINI_PLCC4_3.5x3.5mm_P1.75mm, F.Cu at (393.4, 64.3)
- added D46: SK6812MINI, LED_SMD:LED_SK6812MINI_PLCC4_3.5x3.5mm_P1.75mm, F.Cu at (393.4, 69.4)
- added D47: SK6812MINI, LED_SMD:LED_SK6812MINI_PLCC4_3.5x3.5mm_P1.75mm, F.Cu at (393.4, 74.6)
- added D48: SK6812MINI, LED_SMD:LED_SK6812MINI_PLCC4_3.5x3.5mm_P1.75mm, F.Cu at (393.4, 79.7)
- added D49: SK6812MINI, LED_SMD:LED_SK6812MINI_PLCC4_3.5x3.5mm_P1.75mm, F.Cu at (400.2, 54.1)
- added D50: SK6812MINI, LED_SMD:LED_SK6812MINI_PLCC4_3.5x3.5mm_P1.75mm, F.Cu at (400.2, 59.2)
- added D51: SK6812MINI, LED_SMD:LED_SK6812MINI_PLCC4_3.5x3.5mm_P1.75mm, F.Cu at (400.2, 64.3)
- added D52: SK6812MINI, LED_SMD:LED_SK6812MINI_PLCC4_3.5x3.5mm_P1.75mm, F.Cu at (400.2, 69.4)
- added D53: SK6812MINI, LED_SMD:LED_SK6812MINI_PLCC4_3.5x3.5mm_P1.75mm, F.Cu at (400.2, 74.6)
- added D54: SK6812MINI, LED_SMD:LED_SK6812MINI_PLCC4_3.5x3.5mm_P1.75mm, F.Cu at (400.2, 79.7)
- added D55: SK6812MINI, LED_SMD:LED_SK6812MINI_PLCC4_3.5x3.5mm_P1.75mm, F.Cu at (406.9, 54.1)
- added D56: SK6812MINI, LED_SMD:LED_SK6812MINI_PLCC4_3.5x3.5mm_P1.75mm, F.Cu at (406.9, 59.2)
- added D57: SK6812MINI, LED_SMD:LED_SK6812MINI_PLCC4_3.5x3.5mm_P1.75mm, F.Cu at (406.9, 64.3)
- added D58: SK6812MINI, LED_SMD:LED_SK6812MINI_PLCC4_3.5x3.5mm_P1.75mm, F.Cu at (406.9, 69.4)
- added D59: SK6812MINI, LED_SMD:LED_SK6812MINI_PLCC4_3.5x3.5mm_P1.75mm, F.Cu at (406.9, 74.6)
- added D60: SK6812MINI, LED_SMD:LED_SK6812MINI_PLCC4_3.5x3.5mm_P1.75mm, F.Cu at (406.9, 79.7)
- added D61: SK6812MINI, LED_SMD:LED_SK6812MINI_PLCC4_3.5x3.5mm_P1.75mm, F.Cu at (413.6, 54.1)
- added D62: SK6812MINI, LED_SMD:LED_SK6812MINI_PLCC4_3.5x3.5mm_P1.75mm, F.Cu at (413.6, 59.2)
- added D63: SK6812MINI, LED_SMD:LED_SK6812MINI_PLCC4_3.5x3.5mm_P1.75mm, F.Cu at (413.6, 64.3)
- added D64: SK6812MINI, LED_SMD:LED_SK6812MINI_PLCC4_3.5x3.5mm_P1.75mm, F.Cu at (413.6, 69.4)
- added D65: SK6812MINI, LED_SMD:LED_SK6812MINI_PLCC4_3.5x3.5mm_P1.75mm, F.Cu at (413.6, 74.6)
- added D66: SK6812MINI, LED_SMD:LED_SK6812MINI_PLCC4_3.5x3.5mm_P1.75mm, F.Cu at (413.6, 79.7)
- added D67: SK6812MINI, LED_SMD:LED_SK6812MINI_PLCC4_3.5x3.5mm_P1.75mm, F.Cu at (420.3, 54.1)
- added D68: SK6812MINI, LED_SMD:LED_SK6812MINI_PLCC4_3.5x3.5mm_P1.75mm, F.Cu at (420.3, 59.2)
- added D69: SK6812MINI, LED_SMD:LED_SK6812MINI_PLCC4_3.5x3.5mm_P1.75mm, F.Cu at (420.3, 64.3)
- added D7: SK6812MINI, LED_SMD:LED_SK6812MINI_PLCC4_3.5x3.5mm_P1.75mm, F.Cu at (386.7, 59.2)
- added D70: SK6812MINI, LED_SMD:LED_SK6812MINI_PLCC4_3.5x3.5mm_P1.75mm, F.Cu at (420.3, 69.4)
- added D71: SK6812MINI, LED_SMD:LED_SK6812MINI_PLCC4_3.5x3.5mm_P1.75mm, F.Cu at (420.3, 74.6)
- added D72: SK6812MINI, LED_SMD:LED_SK6812MINI_PLCC4_3.5x3.5mm_P1.75mm, F.Cu at (420.3, 79.7)
- added RSW1: SW_PUSH, Button_Switch_SMD:SW_SPST_TS-1088-xR020, F.Cu at (421.3, 109.5)
- added RSW2: SW_PUSH, Button_Switch_SMD:SW_SPST_TS-1088-xR020, F.Cu at (421.3, 114.1)
- added SW23: SW_PUSH, kbd:ChocV1_V2_Hotswap, F.Cu at (341.7, 57.8)
- added SW24: SW_PUSH, kbd:ChocV1_V2_Hotswap, F.Cu at (341.7, 72.8)
- added SW25: SW_PUSH, kbd:ChocV1_V2_Hotswap, F.Cu at (341.7, 87.9)
- added SW26: SW_PUSH, kbd:ChocV1_V2_Hotswap, F.Cu at (341.7, 102.9)
- added SW27: SW_PUSH, kbd:ChocV1_V2_Hotswap, F.Cu at (341.7, 118.0)
- added SW29: SW_PUSH, kbd:ChocV1_V2_Hotswap, F.Cu at (341.7, 133.0)
- added SW30: SW_PUSH, kbd:ChocV1_V2_Hotswap, F.Cu at (359.0, 57.8)
- added SW31: SW_PUSH, kbd:ChocV1_V2_Hotswap, F.Cu at (359.0, 72.8)
- added SW32: SW_PUSH, kbd:ChocV1_V2_Hotswap, F.Cu at (359.0, 87.9)
- added SW33: SW_PUSH, kbd:ChocV1_V2_Hotswap, F.Cu at (359.0, 102.9)
- added SW35: SW_PUSH, kbd:ChocV1_V2_Hotswap, F.Cu at (359.0, 118.0)
- added SW36: SW_PUSH, kbd:ChocV1_V2_Hotswap, F.Cu at (359.0, 133.0)
- added SW37: SW_PUSH, kbd:ChocV1_V2_Hotswap, F.Cu at (376.2, 57.8)
- added SW38: SW_PUSH, kbd:ChocV1_V2_Hotswap, F.Cu at (376.2, 72.8)
- added SW39: SW_PUSH, kbd:ChocV1_V2_Hotswap, F.Cu at (376.2, 87.9)
- added SW40: SW_PUSH, kbd:ChocV1_V2_Hotswap, F.Cu at (376.2, 102.9)
- added SW41: SW_PUSH, kbd:ChocV1_V2_Hotswap, F.Cu at (376.2, 118.0)
- added SW42: SW_PUSH, kbd:ChocV1_V2_Hotswap, F.Cu at (376.2, 133.0)
- added U1: nice_nano, Library:nice_nano, F.Cu at (401.8, 91.8)
- added U2: nice_nano, Library:nice_nano, F.Cu at (401.8, 111.0)
- added battery1: Conn_01x02_Pin, Connector_JST:JST_SH_BM02B-SRSS-TB_1x02-1MP_P1.00mm_Vertical, F.Cu at (421.2, 85.4)
- added battery2: Conn_01x02_Pin, Connector_JST:JST_SH_BM02B-SRSS-TB_1x02-1MP_P1.00mm_Vertical, F.Cu at (421.2, 91.6)
- added switch1: Conn_01x02_Pin, Connector_JST:JST_SH_BM02B-SRSS-TB_1x02-1MP_P1.00mm_Vertical, F.Cu at (421.2, 97.9)
- added switch2: Conn_01x02_Pin, Connector_JST:JST_SH_BM02B-SRSS-TB_1x02-1MP_P1.00mm_Vertical, F.Cu at (421.2, 104.1)
- D10, D11, D12, D14, D15, D16, D17, D18, D19, D2, D20, D21, D3, D4, D5, D6, D8, D9: footprint kbd:D3_TH_SMD -> Diode_SMD:D_SOD-323_HandSoldering
- SW10, SW11, SW12, SW14, SW15, SW16, SW17, SW18, SW19, SW2, SW20, SW21, SW3, SW4, SW5, SW6, SW8, SW9: footprint keyswitches:Kailh_socket_PG1350_reversible -> kbd:ChocV1_V2_Hotswap
Connections:
- SW10 pad 1: col3 -> col2
- SW11 pad 1: col4 -> col3
- SW12 pad 1: col5 -> col4
- SW14 pad 1: col1 -> col0
- SW15 pad 1: col2 -> col1
- SW16 pad 1: col3 -> col2
- SW17 pad 1: col4 -> col3
- SW18 pad 1: col5 -> col4
- SW19 pad 1: col3 -> col2
- SW2 pad 1: col1 -> col0
- SW20 pad 1: col4 -> col3
- SW21 pad 1: col5 -> col4
- SW3 pad 1: col2 -> col1
- SW4 pad 1: col3 -> col2
- SW5 pad 1: col4 -> col3
- SW6 pad 1: col5 -> col4
- SW8 pad 1: col1 -> col0
- SW9 pad 1: col2 -> col1
Routing:
- net col0: track 15.4 -> 104.9 mm, vias 1 -> 6
- net col4: track 136.4 -> 220.5 mm, vias 8 -> 13
- net col1: track 205.3 -> 262.4 mm, vias 8 -> 10
- net col2: track 151.4 -> 205.1 mm, vias 4 -> 7
- net col3: track 167.9 -> 212.1 mm, vias 7 -> 10
- net Net-(D19-Pad2): track 0.00 -> 41.0 mm, vias 0 -> 1
- net Net-(D19-A): track 41.0 -> 0.00 mm, vias 1 -> 0
- net Net-(D11-Pad2): track 0.00 -> 36.9 mm, vias 0 -> 1
- net Net-(D20-Pad2): track 0.00 -> 36.8 mm, vias 0 -> 2
- net Net-(D20-A): track 36.8 -> 0.00 mm, vias 2 -> 0
- net Net-(D17-A): track 38.0 -> 2.03 mm, vias 2 -> 0
- net Net-(D12-A): track 36.7 -> 2.03 mm, vias 2 -> 0
- net Net-(D16-A): track 36.7 -> 2.03 mm, vias 2 -> 0
- net Net-(D4-A): track 36.4 -> 2.04 mm, vias 2 -> 0
- net Net-(D8-A): track 36.3 -> 2.03 mm, vias 2 -> 0
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
Commit message: feat: update
Parts:
- removed C19, C20, C21, C22, C23, C24, C25, C26, C27, C28, C29, C30, C31, C32, C33, C34, C35, C36: 100nF, Capacitor_SMD:C_0805_2012Metric_Pad1.18x1.45mm_HandSolder
- removed Cap100nf2: C, Capacitor_SMD:C_0805_2012Metric_Pad1.18x1.45mm_HandSolder
- removed D19, D20, D21, D23, D24, D25, D26, D27, D29, D30, D31, D32, D33, D35, D36, D37, D38, D39, D40, D41, D42: D, Diode_SMD:D_SOD-323_HandSoldering
- removed D55, D56, D57, D58, D59, D60, D61, D62, D63, D64, D65, D66, D67, D68, D69, D70, D71, D72: SK6812MINI, LED_SMD:LED_SK6812MINI_PLCC4_3.5x3.5mm_P1.75mm
- removed J1: MJ-4PP-9, kbd:MJ-4PP-9
- removed J2: OLED, foostan:OLED
- removed J3: Conn_01x02_Female, kbd:Battery_TH
- removed JP6, JP61: SDA, foostan:Jumper
- removed JP61, JP62: RAW, foostan:Jumper
- removed JP62, JP68: GND, foostan:Jumper
- removed JP63, JP66: SCL, foostan:Jumper
- removed JP64, JP65: VCC, foostan:Jumper
- removed the RSW1 at (182.8, 93.9)
- removed RSW2: SW_PUSH, Button_Switch_SMD:SW_SPST_TS-1088-xR020
- removed SW19, SW20, SW21, SW23, SW24, SW25, SW26, SW27, SW29, SW30, SW31, SW32, SW33, SW35, SW36, SW37, SW38, SW39, SW40, SW41, SW42: SW_PUSH, kbd:ChocV1_V2_Hotswap
- removed the SW2 at (85.9, 70.4)
- removed the SW2 at (178.2, 55.9)
- removed the U1 at (178.5, 72.1)
- removed the U1 at (401.8, 91.8)
- removed U2: nice_nano, Library:nice_nano
- removed battery2, switch2: Conn_01x02_Pin, Connector_JST:JST_SH_BM02B-SRSS-TB_1x02-1MP_P1.00mm_Vertical
- removed h2: h2, kbd:LEGO_HOLE
- removed h3: h3, kbd:LEGO_HOLE
- removed h4: h4, kbd:LEGO_HOLE
- removed h5: h5, kbd:LEGO_HOLE
- removed h6: h6, kbd:LEGO_HOLE
- removed h7: h7, kbd:LEGO_HOLE
- added D1: D, Diode_SMD:D_SOD-323_HandSoldering, F.Cu at (94.8, 71.0)
- added D13: D, Diode_SMD:D_SOD-323_HandSoldering, F.Cu at (131.0, 86.5)
- added D7: D, Diode_SMD:D_SOD-323_HandSoldering, F.Cu at (112.8, 75.8)
- added H2: MountingHole, MountingHole:MountingHole_2.2mm_M2_DIN965_Pad, F.Cu at (95.0, 83.8)
- added H3: MountingHole, MountingHole:MountingHole_2.2mm_M2_DIN965_Pad, F.Cu at (149.0, 69.8)
- added H4: MountingHole, MountingHole:MountingHole_2.2mm_M2_DIN965_Pad, F.Cu at (124.0, 104.1)
- added H5: MountingHole, MountingHole:MountingHole_2.2mm_M2_DIN965_Pad, F.Cu at (171.3, 96.9)
- added H6: MountingHole, MountingHole:MountingHole_2.2mm_M2_DIN965_Pad, F.Cu at (167.0, 110.4)
- added H7: MountingHole, MountingHole:MountingHole_2.2mm_M2_DIN965_Pad, F.Cu at (185.4, 106.4)
- added SW13: SW_PUSH, keyswitches:Kailh_socket_PG1350_reversible, F.Cu at (121.9, 86.4)
- added SW2: SW_PUSH, keyswitches:Kailh_socket_PG1350_reversible, F.Cu at (103.9, 58.4)
- added SW7: SW_PUSH, keyswitches:Kailh_socket_PG1350_reversible, F.Cu at (103.9, 75.4)
- added U1: nice_nano, Library:nice_nano, F.Cu at (176.6, 73.3)
- C1, C10, C11, C12, C13, C14, C15, C16, C17, C18, C2, C3, C4, C5, C6, C7, C8, C9: value 100nF -> Cap100nf
- Cap100nf1: value C -> C_general
- H1: value h1 -> MountingHole; footprint kbd:LEGO_HOLE -> MountingHole:MountingHole_2.2mm_M2_DIN965_Pad
- LED1: renamed from D7; footprint LED_SMD:LED_SK6812MINI_PLCC4_3.5x3.5mm_P1.75mm -> kbd:YS-SK6812MINI-E
- LED10: renamed from D46; footprint LED_SMD:LED_SK6812MINI_PLCC4_3.5x3.5mm_P1.75mm -> kbd:YS-SK6812MINI-E
- LED11: renamed from D47; footprint LED_SMD:LED_SK6812MINI_PLCC4_3.5x3.5mm_P1.75mm -> kbd:YS-SK6812MINI-E
- LED12: renamed from D48; footprint LED_SMD:LED_SK6812MINI_PLCC4_3.5x3.5mm_P1.75mm -> kbd:YS-SK6812MINI-E
- LED13: renamed from D49; footprint LED_SMD:LED_SK6812MINI_PLCC4_3.5x3.5mm_P1.75mm -> kbd:YS-SK6812MINI-E
- LED14: renamed from D50; footprint LED_SMD:LED_SK6812MINI_PLCC4_3.5x3.5mm_P1.75mm -> kbd:YS-SK6812MINI-E
- LED15: renamed from D51; footprint LED_SMD:LED_SK6812MINI_PLCC4_3.5x3.5mm_P1.75mm -> kbd:YS-SK6812MINI-E
- LED16: renamed from D52; footprint LED_SMD:LED_SK6812MINI_PLCC4_3.5x3.5mm_P1.75mm -> kbd:YS-SK6812MINI-E
- LED17: renamed from D53; footprint LED_SMD:LED_SK6812MINI_PLCC4_3.5x3.5mm_P1.75mm -> kbd:YS-SK6812MINI-E
- LED18: renamed from D54; footprint LED_SMD:LED_SK6812MINI_PLCC4_3.5x3.5mm_P1.75mm -> kbd:YS-SK6812MINI-E
- LED2: renamed from D1; footprint LED_SMD:LED_SK6812MINI_PLCC4_3.5x3.5mm_P1.75mm -> kbd:YS-SK6812MINI-E
- LED3: renamed from D13; footprint LED_SMD:LED_SK6812MINI_PLCC4_3.5x3.5mm_P1.75mm -> kbd:YS-SK6812MINI-E
- LED4: renamed from D22; footprint LED_SMD:LED_SK6812MINI_PLCC4_3.5x3.5mm_P1.75mm -> kbd:YS-SK6812MINI-E
- LED5: renamed from D28; footprint LED_SMD:LED_SK6812MINI_PLCC4_3.5x3.5mm_P1.75mm -> kbd:YS-SK6812MINI-E
- LED6: renamed from D34; footprint LED_SMD:LED_SK6812MINI_PLCC4_3.5x3.5mm_P1.75mm -> kbd:YS-SK6812MINI-E
- LED7: renamed from D43; footprint LED_SMD:LED_SK6812MINI_PLCC4_3.5x3.5mm_P1.75mm -> kbd:YS-SK6812MINI-E
- LED8: renamed from D44; footprint LED_SMD:LED_SK6812MINI_PLCC4_3.5x3.5mm_P1.75mm -> kbd:YS-SK6812MINI-E
- LED9: renamed from D45; footprint LED_SMD:LED_SK6812MINI_PLCC4_3.5x3.5mm_P1.75mm -> kbd:YS-SK6812MINI-E
- SW1: value SW_SPDT -> SW_PUSH; footprint Buttons_Switches:SW_SPDT+H-MSK12C01_hor(7pin_SMD) -> keyswitches:Kailh_socket_PG1350_reversible
- SW10, SW11, SW12, SW14, SW15, SW16, SW17, SW18, SW3, SW4, SW5, SW6, SW8, SW9: footprint kbd:ChocV1_V2_Hotswap -> keyswitches:Kailh_socket_PG1350_reversible
- moved LED11 308.5 mm to (86.0, 99.8)
- moved LED1 300.8 mm to (86.0, 65.8)
- moved LED6 300.7 mm to (86.0, 82.8)
- moved C6 298.1 mm to (90.5, 96.0)
- moved C11 297.7 mm to (94.8, 94.5), turned to -90 degrees
- moved C1 294.4 mm to (94.8, 77.5), turned to -90 degrees
- moved LED7 289.9 mm to (104.0, 70.8)
- moved LED12 289.6 mm to (104.0, 87.8)
- moved LED2 282.7 mm to (104.0, 53.7)
- moved C2 282.0 mm to (112.8, 54.5), turned to -90 degrees
- moved C7 281.5 mm to (112.8, 71.8), turned to -90 degrees
- moved C12 281.1 mm to (112.8, 88.2), turned to -90 degrees
- moved LED13 279.5 mm to (122.0, 81.8)
- moved LED8 271.8 mm to (121.8, 64.8)
- moved LED16 270.5 mm to (134.0, 117.8), turned to 180 degrees
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Connections:
- D11 pad 1: row1 -> row2
- D12 pad 1: row1 -> row2
- D16 pad 1: row2 -> row3
- D17 pad 1: row2 -> row3
- D18 pad 1: row2 -> row3
- D6 pad 1: row0 -> row1
- LED1 pad 3: LED -> Net-(LED1-DIN)
- LED10 pad 1: LED_bis -> Net-(LED10-DOUT)
- LED11 pad 3: LED_bis -> Net-(LED11-DIN)
- LED15 pad 1: Net-(D51-DOUT) -> Net-(LED10-DOUT)
- LED16 pad 3: Net-(D51-DOUT) -> Net-(LED11-DIN)
- LED5 pad 1: Net-(D28-DOUT) -> LED
- LED6 pad 3: Net-(D28-DOUT) -> Net-(LED1-DIN)
- SW1 pad 1: (no net) -> col0
- SW10 pad 1: col2 -> col4
- SW11 pad 1: col3 -> col0
- SW12 pad 1: col4 -> col1
- SW14 pad 1: col0 -> col3
- SW15 pad 1: col1 -> col4
- SW3 pad 1: col1 -> col2
- SW4 pad 1: col2 -> col3
- SW5 pad 1: col3 -> col4
- SW6 pad 1: col4 -> col0
- SW8 pad 1: col0 -> col2
- SW9 pad 1: col1 -> col3
Routing:
- net col1: track 262.4 -> 145.0 mm, vias 10 -> 5
- net col5: track 106.6 -> 0.00 mm, vias 5 -> 0
- net col4: track 220.5 -> 116.5 mm, vias 13 -> 4
- net col0: track 104.9 -> 181.1 mm, vias 6 -> 7
- net SCL: track 66.3 -> 0.00 mm, vias 4 -> 0
- net Net-(LED11-DIN): track 0.00 -> 63.2 mm, vias 0 -> 2
- net data: track 62.7 -> 0.00 mm
- net col3: track 212.1 -> 151.8 mm, vias 10 -> 7
- net SDA: track 59.2 -> 0.00 mm, vias 2 -> 0
- net col2: track 205.1 -> 151.7 mm, vias 7 -> 14
- net row3: track 123.2 -> 70.2 mm, vias 3 -> 0
- net row0: track 155.4 -> 105.8 mm, vias 2 -> 0
- net row2: track 156.9 -> 109.6 mm, vias 3 -> 0
- net BAT: track 0.00 -> 43.1 mm, vias 0 -> 2
- net row1: track 136.5 -> 95.3 mm, vias 1 -> 0
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- added copper zone on F.Cu, net GND
- added copper zone on B.Cu, net VCC
- removed copper zone on B.Cu, net (none)
- removed copper zone on F.Cu, net (none)
Other:
- board text added: "${REFERENCE}"
- board text removed: "GND"
- board text removed: "chocofi @pashutk"

Commit message: feat: cilose
Parts:
- moved D6 15.9 mm to (81.2, 96.0), turned to 0 degrees
- moved D1 15.5 mm to (81.5, 79.0), turned to 0 degrees
- moved C4 13.1 mm to (144.5, 67.5), turned to 0 degrees
- moved RSW1 9.51 mm to (184.5, 100.5), turned to -90 degrees
- moved D3 7.25 mm to (131.0, 60.0)
- moved switch1 4.74 mm to (184.5, 92.5), turned to 90 degrees
- moved battery1 4.66 mm to (177.7, 92.5), turned to 90 degrees
- moved C1 4.51 mm to (90.5, 79.0), turned to 0 degrees
- moved C9 4.42 mm to (144.5, 84.5), turned to 0 degrees
- moved C3 4.27 mm to (127.0, 61.0), turned to 0 degrees
- moved Cap100nf1 3.54 mm to (178.0, 100.5)
- moved U1 2.04 mm to (178.0, 71.8)
- moved C7 1.77 mm to (113.0, 70.0)
- moved D4 1.75 mm to (149.0, 57.5)
- moved C2 1.52 mm to (113.0, 53.0)
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Routing:
- net VCC: track 78.2 -> 36.0 mm, vias 23 -> 22
- net col1: track 145.0 -> 174.8 mm, vias 5 -> 10
- net row0: track 105.8 -> 133.0 mm, vias 0 -> 1
- net col2: track 151.7 -> 175.6 mm, vias 14 -> 9
- net row1: track 95.3 -> 114.8 mm, vias 0 -> 1
- net Net-(D18-A): track 42.2 -> 23.5 mm, vias 1 -> 2
- net Net-(D16-A): track 37.5 -> 22.1 mm, vias 1 -> 2
- net Net-(LED3-VSS): track 13.7 -> 27.0 mm
- net GND: track 95.0 -> 82.5 mm, vias 25 -> 16
- net col3: track 151.8 -> 162.7 mm, vias 7 -> 9
- net Net-(LED4-VSS): track 7.37 -> 17.6 mm, vias 2 -> 3
- net Net-(LED16-VSS): track 27.7 -> 19.2 mm, vias 2 -> 0
- net Net-(D3-A): track 22.6 -> 30.3 mm, vias 1 -> 4
- net reset: track 44.5 -> 37.0 mm
- net LED: track 18.6 -> 11.4 mm, vias 1 -> 0
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
Commit message: feat: wip1
Parts:
- added Right: nice_nano, Library:nice_nano, B.Cu at (178.8, 73.0)
- moved D2 16.5 mm to (99.5, 67.0), turned to 0 degrees
- moved D7 16.3 mm to (99.8, 84.0), turned to 0 degrees
- moved C2 14.8 mm to (108.2, 67.0), turned to 0 degrees
- moved C7 14.8 mm to (108.2, 84.0), turned to 0 degrees
- moved C8 14.3 mm to (126.2, 78.0), turned to 0 degrees
- moved D3 13.3 mm to (117.8, 61.0), turned to 0 degrees
- moved D13 11.5 mm to (127.0, 96.8)
- moved C11 6.75 mm to (95.0, 87.8)
- moved D12 6.04 mm to (115.5, 97.5)
- moved C13 3.25 mm to (131.0, 84.8)
- moved Left 1.25 mm to (176.8, 71.8)
- moved C12 1.00 mm to (113.0, 86.5)
- renumbered U1 to Left
Routing:
- net GND: track 82.5 -> 5.07 mm, vias 16 -> 0
- net col4: track 122.8 -> 148.7 mm, vias 5 -> 8
- net unconnected-(U1-P1.06-Pad12): track 0.00 -> 17.8 mm
- net unconnected-(U1-P1.04-Pad11): track 0.00 -> 17.8 mm
- net nice!view_MOSI: track 0.00 -> 17.8 mm
- net nice!view_CSL: track 0.00 -> 17.8 mm
- net nice!view_CS: track 0.00 -> 17.8 mm
- net LED: track 11.4 -> 27.9 mm
- net reset: track 37.0 -> 53.4 mm
- net BAT: track 47.8 -> 62.7 mm, vias 0 -> 1
- net row3: track 74.9 -> 89.2 mm
- net Net-(LED3-VSS): track 27.0 -> 13.1 mm, vias 2 -> 1
- net unconnected-(U1-P1.11-Pad15): track 0.00 -> 13.8 mm
- net unconnected-(U1-NFC2/P0.10-Pad14): track 0.00 -> 13.8 mm
- net unconnected-(U1-NFC1/P0.09-Pad13): track 0.00 -> 13.8 mm
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Other:
- copper layers 2 -> 4

Commit message: feat: update
Routing:
- net GND: track 5.07 -> 150.3 mm, vias 0 -> 27
- net VCC: track 25.7 -> 82.0 mm, vias 19 -> 17
- net col3: track 174.5 -> 130.5 mm, vias 8 -> 4
- net Net-(LED4-DOUT): track 14.1 -> 53.6 mm, vias 0 -> 1
- net Net-(LED8-DOUT): track 16.1 -> 49.2 mm, vias 0 -> 1
- net Net-(LED13-DOUT): track 15.6 -> 46.1 mm, vias 0 -> 2
- net Net-(LED3-DOUT): track 18.0 -> 48.5 mm, vias 0 -> 1
- net col2: track 185.2 -> 155.2 mm, vias 10 -> 4
- net Net-(LED14-DOUT): track 14.3 -> 43.2 mm, vias 0 -> 1
- net Net-(LED2-DOUT): track 14.4 -> 42.6 mm, vias 0 -> 1
- net Net-(LED12-DOUT): track 14.4 -> 42.1 mm, vias 0 -> 2
- net Net-(LED11-DOUT): track 16.9 -> 43.2 mm, vias 0 -> 3
- net Net-(LED7-DOUT): track 14.2 -> 40.2 mm, vias 0 -> 1
- net col4: track 148.7 -> 123.3 mm, vias 8 -> 4
- net Net-(LED3-VSS): track 13.1 -> 38.4 mm, vias 1 -> 3
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