File: pcb/chocofi.kicad_pcb (KiCad board)
At the start: 4 copper layers, 111.3 x 90 mm, 85 parts, among them SW1 SW_PUSH, SW10 SW_PUSH, SW11 SW_PUSH, SW12 SW_PUSH, SW13 SW_PUSH, SW14 SW_PUSH, SW15 SW_PUSH, SW16 SW_PUSH, SW17 SW_PUSH, SW18 SW_PUSH, SW2 SW_PUSH, SW3 SW_PUSH, SW4 SW_PUSH, SW5 SW_PUSH, SW6 SW_PUSH, SW7 SW_PUSH, SW8 SW_PUSH, SW9 SW_PUSH

Commit message: wip(pcb): update it
Parts:
- added nice!view1: Conn_01x05_MountingPin, Connector_PinHeader_2.54mm:PinHeader_1x05_P2.54mm_Vertical, F.Cu at (48.8, 49.1)
- SW1, SW18, SW8: footprint keyswitches:Kailh_socket_PG1350_reversible -> PCM_Switch_Keyboard_Hotswap_Kailh:SW_Hotswap_Kailh_Choc_V1V2_Plated
- SW10: renamed from SW16; footprint keyswitches:Kailh_socket_PG1350_reversible -> PCM_Switch_Keyboard_Hotswap_Kailh:SW_Hotswap_Kailh_Choc_V1V2_Plated
- SW11: renamed from SW4; footprint keyswitches:Kailh_socket_PG1350_reversible -> PCM_Switch_Keyboard_Hotswap_Kailh:SW_Hotswap_Kailh_Choc_V1V2_Plated
- SW12: renamed from SW9; footprint keyswitches:Kailh_socket_PG1350_reversible -> PCM_Switch_Keyboard_Hotswap_Kailh:SW_Hotswap_Kailh_Choc_V1V2_Plated
- SW13: renamed from SW14; footprint keyswitches:Kailh_socket_PG1350_reversible -> PCM_Switch_Keyboard_Hotswap_Kailh:SW_Hotswap_Kailh_Choc_V1V2_Plated
- SW14: renamed from SW17; footprint keyswitches:Kailh_socket_PG1350_reversible -> PCM_Switch_Keyboard_Hotswap_Kailh:SW_Hotswap_Kailh_Choc_V1V2_Plated
- SW15: renamed from SW5; footprint keyswitches:Kailh_socket_PG1350_reversible -> PCM_Switch_Keyboard_Hotswap_Kailh:SW_Hotswap_Kailh_Choc_V1V2_Plated
- SW16: renamed from SW10; footprint keyswitches:Kailh_socket_PG1350_reversible -> PCM_Switch_Keyboard_Hotswap_Kailh:SW_Hotswap_Kailh_Choc_V1V2_Plated
- SW17: renamed from SW15; footprint keyswitches:Kailh_socket_PG1350_reversible -> PCM_Switch_Keyboard_Hotswap_Kailh:SW_Hotswap_Kailh_Choc_V1V2_Plated
- SW2: renamed from SW6; footprint keyswitches:Kailh_socket_PG1350_reversible -> PCM_Switch_Keyboard_Hotswap_Kailh:SW_Hotswap_Kailh_Choc_V1V2_Plated
- SW3: renamed from SW11; footprint keyswitches:Kailh_socket_PG1350_reversible -> PCM_Switch_Keyboard_Hotswap_Kailh:SW_Hotswap_Kailh_Choc_V1V2_Plated
- SW4: renamed from SW2; footprint keyswitches:Kailh_socket_PG1350_reversible -> PCM_Switch_Keyboard_Hotswap_Kailh:SW_Hotswap_Kailh_Choc_V1V2_Plated
- SW5: renamed from SW7; footprint keyswitches:Kailh_socket_PG1350_reversible -> PCM_Switch_Keyboard_Hotswap_Kailh:SW_Hotswap_Kailh_Choc_V1V2_Plated
- SW6: renamed from SW12; footprint keyswitches:Kailh_socket_PG1350_reversible -> PCM_Switch_Keyboard_Hotswap_Kailh:SW_Hotswap_Kailh_Choc_V1V2_Plated
- SW7: renamed from SW3; footprint keyswitches:Kailh_socket_PG1350_reversible -> PCM_Switch_Keyboard_Hotswap_Kailh:SW_Hotswap_Kailh_Choc_V1V2_Plated
- SW9: renamed from SW13; footprint keyswitches:Kailh_socket_PG1350_reversible -> PCM_Switch_Keyboard_Hotswap_Kailh:SW_Hotswap_Kailh_Choc_V1V2_Plated
- moved LED18 157.6 mm to (42.0, 42.6), turned to 0 degrees
- moved C18 140.6 mm to (58.5, 36.3)
- moved LED17 137.9 mm to (42.0, 37.8), turned to 0 degrees
- moved LED5 134.2 mm to (24.2, 47.5)
- moved LED15 131.8 mm to (42.0, 28.2)
- moved LED10 130.0 mm to (33.1, 37.8)
- moved C17 128.0 mm to (58.5, 33.3)
- moved C15 125.6 mm to (58.5, 27.3), turned to 0 degrees
- moved LED16 125.1 mm to (42.0, 33.0), turned to 0 degrees
- moved C10 120.2 mm to (53.7, 33.3), turned to 0 degrees
- moved C5 119.4 mm to (48.9, 39.3), turned to 0 degrees
- moved LED4 116.4 mm to (24.2, 42.6)
- moved LED9 113.6 mm to (33.1, 33.0)
- moved LED14 111.2 mm to (33.1, 57.1)
- moved C16 109.0 mm to (58.5, 30.3)
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- renumbered D16 to D10, D4 to D11, D9 to D12, D14 to D13, D17 to D14, D5 to D15, D10 to D16, D15 to D17, D6 to D2, D11 to D3, D2 to D4, D7 to D5, D12 to D6, D3 to D7, D13 to D9, Left to U1, Right to U1
Connections:
- C1 pad 1: Net-(LED1-VSS) -> VCC
- C1 pad 2: VCC -> Net-(LED1-VDD)
- C10 pad 1: Net-(LED10-VSS) -> VCC
- C10 pad 2: VCC -> Net-(LED10-VDD)
- C11 pad 1: Net-(LED11-VSS) -> VCC
- C11 pad 2: VCC -> Net-(LED11-VDD)
- C12 pad 1: Net-(LED12-VSS) -> Net-(C12-Pad1)
- C12 pad 2: VCC -> Net-(LED12-VDD)
- C13 pad 1: Net-(LED13-VSS) -> VCC
- C13 pad 2: VCC -> Net-(LED13-VDD)
- C14 pad 1: Net-(LED14-VSS) -> VCC
- C14 pad 2: VCC -> Net-(LED14-VDD)
- C15 pad 1: Net-(LED15-VSS) -> VCC
- C15 pad 2: VCC -> Net-(LED15-VDD)
- C16 pad 1: Net-(LED16-VSS) -> VCC
- C16 pad 2: VCC -> Net-(LED16-VDD)
- C17 pad 1: Net-(LED17-VSS) -> VCC
- C17 pad 2: VCC -> Net-(LED17-VDD)
- C18 pad 1: Net-(LED18-VSS) -> Net-(C12-Pad1)
- C18 pad 2: VCC -> Net-(LED18-VDD)
- C2 pad 1: Net-(LED2-VSS) -> VCC
- C2 pad 2: VCC -> Net-(LED2-VDD)
- C3 pad 1: Net-(LED3-VSS) -> Net-(C12-Pad1)
- C3 pad 2: VCC -> Net-(LED3-VDD)
- C4 pad 1: Net-(LED4-VSS) -> VCC
- C4 pad 2: VCC -> Net-(LED4-VDD)
- C5 pad 1: Net-(LED5-VSS) -> Net-(C12-Pad1)
- C5 pad 2: VCC -> Net-(LED5-VDD)
- C6 pad 1: Net-(LED6-VSS) -> VCC
- C6 pad 2: VCC -> Net-(LED6-VDD)
- C7 pad 1: Net-(LED7-VSS) -> VCC
- C7 pad 2: VCC -> Net-(LED7-VDD)
- C8 pad 1: Net-(LED8-VSS) -> Net-(C12-Pad1)
- C8 pad 2: VCC -> Net-(LED8-VDD)
- C9 pad 1: Net-(LED9-VSS) -> VCC
- C9 pad 2: VCC -> Net-(LED9-VDD)
- LED1 pad 2: Net-(LED1-VSS) -> GND
- LED1 pad 3: Net-(LED1-DIN) -> LED
- LED1 pad 4: GND -> Net-(LED1-VDD)
- LED10 pad 2: Net-(LED10-VSS) -> GND
- LED10 pad 4: GND -> Net-(LED10-VDD)
- LED11 pad 2: Net-(LED11-VSS) -> GND
- LED11 pad 4: GND -> Net-(LED11-VDD)
- LED12 pad 2: Net-(LED12-VSS) -> GND
- LED12 pad 3: Net-(LED11-DOUT) -> Net-(LED12-DIN)
- LED12 pad 4: GND -> Net-(LED12-VDD)
- LED13 pad 2: Net-(LED13-VSS) -> GND
- LED13 pad 3: Net-(LED12-DOUT) -> Net-(LED13-DIN)
- LED13 pad 4: GND -> Net-(LED13-VDD)
- LED14 pad 1: Net-(LED14-DOUT) -> Net-(LED10-DIN)
- LED14 pad 2: Net-(LED14-VSS) -> GND
- LED14 pad 3: Net-(LED13-DOUT) -> Net-(LED14-DIN)
- LED14 pad 4: GND -> Net-(LED14-VDD)
- LED15 pad 1: Net-(LED10-DOUT) -> Net-(LED13-DIN)
- LED15 pad 2: Net-(LED15-VSS) -> GND
- LED15 pad 3: Net-(LED14-DOUT) -> Net-(LED15-DIN)
- LED15 pad 4: GND -> Net-(LED15-VDD)
- LED16 pad 2: Net-(LED16-VSS) -> GND
- LED16 pad 3: Net-(LED11-DIN) -> Net-(LED11-DOUT)
- LED16 pad 4: GND -> Net-(LED16-VDD)
- LED17 pad 1: Net-(LED17-DOUT) -> Net-(LED14-DIN)
- LED17 pad 2: Net-(LED17-VSS) -> GND
- LED17 pad 4: GND -> Net-(LED17-VDD)
- LED18 pad 1: unconnected-(LED18-DOUT-Pad1) -> Net-(LED15-DIN)
- LED18 pad 2: Net-(LED18-VSS) -> GND
- LED18 pad 3: Net-(LED17-DOUT) -> Net-(LED12-DOUT)
- LED18 pad 4: GND -> Net-(LED18-VDD)
- LED2 pad 2: Net-(LED2-VSS) -> GND
- LED2 pad 3: Net-(LED1-DOUT) -> Net-(LED2-DIN)
- LED2 pad 4: GND -> Net-(LED2-VDD)
- LED3 pad 2: Net-(LED3-VSS) -> GND
- LED3 pad 4: GND -> Net-(LED3-VDD)
- LED4 pad 2: Net-(LED4-VSS) -> GND
- LED4 pad 3: Net-(LED3-DOUT) -> Net-(LED1-DOUT)
- LED4 pad 4: GND -> Net-(LED4-VDD)
- LED5 pad 1: LED -> Net-(LED5-DOUT)
- LED5 pad 2: Net-(LED5-VSS) -> GND
- LED5 pad 3: Net-(LED4-DOUT) -> Net-(LED3-DOUT)
- LED5 pad 4: GND -> Net-(LED5-VDD)
- LED6 pad 1: Net-(LED6-DOUT) -> Net-(LED2-DIN)
- LED6 pad 2: Net-(LED6-VSS) -> GND
- LED6 pad 3: Net-(LED1-DIN) -> Net-(LED10-DOUT)
- LED6 pad 4: GND -> Net-(LED6-VDD)
- LED7 pad 1: Net-(LED7-DOUT) -> Net-(LED11-DIN)
- LED7 pad 2: Net-(LED7-VSS) -> GND
- LED7 pad 3: Net-(LED6-DOUT) -> Net-(LED4-DOUT)
- LED7 pad 4: GND -> Net-(LED7-VDD)
- LED8 pad 1: Net-(LED8-DOUT) -> Net-(LED12-DIN)
- LED8 pad 2: Net-(LED8-VSS) -> GND
- LED8 pad 3: Net-(LED7-DOUT) -> Net-(LED5-DOUT)
- LED8 pad 4: GND -> Net-(LED8-VDD)
- LED9 pad 1: Net-(LED10-DIN) -> unconnected-(LED9-DOUT-Pad1)
- LED9 pad 2: Net-(LED9-VSS) -> GND
- LED9 pad 3: Net-(LED8-DOUT) -> Net-(LED13-DOUT)
- LED9 pad 4: GND -> Net-(LED9-VDD)
Routing:
- net col0: track 179.8 -> 0.00 mm, vias 3 -> 0
- net col1: track 158.4 -> 0.00 mm, vias 3 -> 0
- net col2: track 155.2 -> 0.00 mm, vias 4 -> 0
- net GND: track 150.3 -> 0.00 mm, vias 27 -> 0
- net col3: track 130.5 -> 0.00 mm, vias 4 -> 0
- net row0: track 129.6 -> 0.00 mm, vias 5 -> 0
- net row1: track 123.6 -> 0.00 mm, vias 5 -> 0
- net col4: track 123.3 -> 0.00 mm, vias 4 -> 0
- net row2: track 112.8 -> 0.00 mm, vias 5 -> 0
- net row3: track 94.5 -> 0.00 mm, vias 3 -> 0
- net VCC: track 82.0 -> 0.00 mm, vias 17 -> 0
- net Net-(LED11-DIN): track 73.1 -> 0.00 mm, vias 2 -> 0
- net BAT: track 67.5 -> 0.00 mm, vias 2 -> 0
- net reset: track 65.2 -> 0.00 mm, vias 1 -> 0
- net Net-(LED4-DOUT): track 53.6 -> 0.00 mm, vias 1 -> 0
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
Commit message: feat(pcb): upgrade
Parts:
- removed Cap100nf1: C_general, Capacitor_SMD:C_0805_2012Metric_Pad1.18x1.45mm_HandSolder
- added C_BAT1: Cap100nf, Capacitor_SMD:C_0805_2012Metric_Pad1.18x1.45mm_HandSolder, F.Cu at (184.6, 96.0)
- added nice!view1: Conn_01x05_MountingPin, Connector_PinHeader_2.54mm:PinHeader_1x05_P2.54mm_Vertical, B.Cu at (184.1, 92.0)
- C1, C10, C11, C12, C13, C14, C15, C16, C17, C18, C2, C3, C4, C5, C6, C7, C8, C9: footprint Capacitor_SMD:C_0805_2012Metric_Pad1.18x1.45mm_HandSolder -> Library:C_0805_2012Metric_Pad1.18x1.45mm_HandSolder_Custom
- D1, D10, D11, D12, D13, D14, D15, D16, D17, D18, D2, D3, D4, D5, D6, D7, D8, D9: footprint Diode_SMD:D_SOD-323_HandSoldering -> Library:D_SOD-323_HandSoldering_Custom
- moved LED18 158.1 mm to (179.1, 121.3), turned to 60 degrees
- moved C18 148.4 mm to (176.0, 127.0), turned to -30 degrees
- moved LED14 135.5 mm to (152.8, 120.5), turned to -15 degrees
- moved nice!view1 130.4 mm to (172.6, 90.0), turned to 90 degrees
- moved LED10 128.9 mm to (133.9, 118.1)
- moved LED17 127.3 mm to (158.0, 90.3)
- moved LED16 122.8 mm to (158.0, 73.3)
- moved LED15 119.2 mm to (157.8, 56.3)
- moved C14 118.7 mm to (146.7, 119.1), turned to -105 degrees
- moved C10 112.8 mm to (127.8, 118.3), turned to -90 degrees
- moved LED13 112.5 mm to (139.8, 87.9)
- moved LED12 109.4 mm to (139.9, 70.9)
- moved C17 109.2 mm to (151.7, 90.1), turned to -90 degrees
- moved LED11 107.4 mm to (139.9, 53.9)
- moved C16 102.7 mm to (151.8, 73.1), turned to -90 degrees
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Connections:
- C12 pad 1: Net-(C12-Pad1) -> VCC
- C18 pad 1: Net-(C12-Pad1) -> VCC
- C3 pad 1: Net-(C12-Pad1) -> VCC
- C5 pad 1: Net-(C12-Pad1) -> VCC
- C8 pad 1: Net-(C12-Pad1) -> VCC
- LED11 pad 3: Net-(LED11-DIN) -> Net-(LED10-DOUT)
- LED12 pad 3: Net-(LED12-DIN) -> Net-(LED11-DOUT)
- LED13 pad 3: Net-(LED13-DIN) -> Net-(LED12-DOUT)
- LED14 pad 1: Net-(LED10-DIN) -> Net-(LED14-DOUT)
- LED14 pad 3: Net-(LED14-DIN) -> Net-(LED13-DOUT)
- LED15 pad 1: Net-(LED13-DIN) -> Net-(LED15-DOUT)
- LED15 pad 3: Net-(LED15-DIN) -> Net-(LED14-DOUT)
- LED16 pad 3: Net-(LED11-DOUT) -> Net-(LED15-DOUT)
- LED17 pad 1: Net-(LED14-DIN) -> Net-(LED17-DOUT)
- LED18 pad 1: Net-(LED15-DIN) -> unconnected-(LED18-DOUT-Pad1)
- LED18 pad 3: Net-(LED12-DOUT) -> Net-(LED17-DOUT)
- LED2 pad 3: Net-(LED2-DIN) -> Net-(LED1-DOUT)
- LED4 pad 3: Net-(LED1-DOUT) -> Net-(LED3-DOUT)
- LED5 pad 3: Net-(LED3-DOUT) -> Net-(LED4-DOUT)
- LED6 pad 1: Net-(LED2-DIN) -> Net-(LED6-DOUT)
- LED6 pad 3: Net-(LED10-DOUT) -> Net-(LED5-DOUT)
- LED7 pad 1: Net-(LED11-DIN) -> Net-(LED7-DOUT)
- LED7 pad 3: Net-(LED4-DOUT) -> Net-(LED6-DOUT)
- LED8 pad 1: Net-(LED12-DIN) -> Net-(LED8-DOUT)
- LED8 pad 3: Net-(LED5-DOUT) -> Net-(LED7-DOUT)
- LED9 pad 1: unconnected-(LED9-DOUT-Pad1) -> Net-(LED10-DIN)
- LED9 pad 3: Net-(LED13-DOUT) -> Net-(LED8-DOUT)
Routing:
- net col0: track 0.00 -> 143.7 mm, vias 0 -> 2
- net col2: track 0.00 -> 134.4 mm, vias 0 -> 1
- net row0: track 0.00 -> 124.2 mm, vias 0 -> 5
- net row2: track 0.00 -> 123.1 mm, vias 0 -> 6
- net col1: track 0.00 -> 120.3 mm, vias 0 -> 3
- net row1: track 0.00 -> 118.9 mm, vias 0 -> 5
- net LED: track 0.00 -> 113.6 mm, vias 0 -> 3
- net col3: track 0.00 -> 111.7 mm, vias 0 -> 1
- net row3: track 0.00 -> 109.7 mm, vias 0 -> 4
- net col4: track 0.00 -> 85.5 mm, vias 0 -> 1
- net Net-(LED14-DOUT): track 0.00 -> 84.1 mm, vias 0 -> 3
- net Net-(LED10-DOUT): track 0.00 -> 81.4 mm, vias 0 -> 3
- net Net-(LED5-DOUT): track 0.00 -> 70.0 mm, vias 0 -> 3
- net Net-(LED17-DOUT): track 0.00 -> 66.2 mm, vias 0 -> 4
- net Net-(LED3-DOUT): track 0.00 -> 66.1 mm, vias 0 -> 3
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
Commit message: feat(pcb): update it
Parts:
- battery1, switch1: footprint Connector_JST:JST_SH_BM02B-SRSS-TB_1x02-1MP_P1.00mm_Vertical -> Library:JST_SH_SM02B-SRSS-TB_1x02-1MP_P1.00mm_Horizontal_Custom
- moved battery1 3.48 mm to (176.0, 106.5)
- moved switch1 1.97 mm to (183.7, 101.0)
Routing:
- net GND: track 60.9 -> 83.1 mm
- net BAT_switch: track 9.20 -> 23.0 mm, vias 0 -> 1
- net reset: track 48.8 -> 53.8 mm
- net BAT: track 61.4 -> 64.5 mm, vias 0 -> 1
- net Net-(LED17-DOUT): track 66.2 -> 67.2 mm

Commit message: feat(pcb): have a good version
Parts:
- C1, C10, C11, C12, C13, C14, C15, C16, C17, C18, C2, C3, C4, C5, C6, C7, C8, C9: footprint Library:C_0805_2012Metric_Pad1.18x1.45mm_HandSolder_Custom -> chocofi:C_0805_2012Metric_Pad1.18x1.45mm_HandSolder
- C_BAT1: footprint Capacitor_SMD:C_0805_2012Metric_Pad1.18x1.45mm_HandSolder -> chocofi:C_0805_2012Metric_Pad1.18x1.45mm_HandSolder
- D1, D10, D11, D12, D13, D14, D15, D16, D17, D18, D2, D3, D4, D5, D6, D7, D8, D9: footprint Library:D_SOD-323_HandSoldering_Custom -> chocofi:D_SOD-323_HandSoldering
- LED1, LED10, LED11, LED12, LED13, LED14, LED15, LED16, LED17, LED18, LED2, LED3, LED4, LED5, LED6, LED7, LED8, LED9: footprint kbd:YS-SK6812MINI-E -> chocofi:YS-SK6812MINI-E
- SW1, SW10, SW11, SW12, SW13, SW14, SW15, SW16, SW17, SW18, SW2, SW3, SW4, SW5, SW6, SW7, SW8, SW9: footprint PCM_Switch_Keyboard_Hotswap_Kailh:SW_Hotswap_Kailh_Choc_V1V2_Plated -> chocofi:SW_Hotswap_Kailh_Choc_V1V2_Plated
- U1 (x2): footprint Library:nice_nano -> chocofi:nice_nano
- battery1, switch1: footprint Library:JST_SH_SM02B-SRSS-TB_1x02-1MP_P1.00mm_Horizontal_Custom -> chocofi:JST_SH_SM02B-SRSS-TB_1x02-1MP_P1.00mm_Horizontal
- nice!view1 (x2): footprint Connector_PinHeader_2.54mm:PinHeader_1x05_P2.54mm_Vertical -> chocofi:PinHeader_1x05_P2.54mm_Vertical
- moved battery1 5.32 mm to (172.0, 103.0), turned to 0 degrees
- moved switch1 4.18 mm to (180.0, 103.0), turned to 0 degrees
- moved LED4 0.53 mm to (103.9, 53.7)
- moved LED13 0.43 mm to (139.9, 88.3)
- moved LED10 0.42 mm to (134.0, 117.7)
- moved LED11 0.42 mm to (139.9, 54.3)
- moved LED12 0.42 mm to (139.9, 71.3)
- moved LED6 0.41 mm to (103.9, 87.7)
- moved LED15 0.41 mm to (157.9, 56.7)
- moved LED16 0.41 mm to (157.9, 73.7)
- moved LED17 0.41 mm to (157.9, 90.7)
- moved LED2 0.41 mm to (85.9, 82.7)
- moved LED8 0.41 mm to (121.9, 64.7)
- moved LED9 0.41 mm to (121.9, 81.7)
- moved LED18 0.40 mm to (178.7, 121.1)
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Routing:
- net col1: track 120.3 -> 169.5 mm, vias 3 -> 5
- net GND: track 83.1 -> 34.2 mm, vias 22 -> 20
- net col0: track 143.7 -> 192.4 mm, vias 2 -> 5
- net col4: track 85.5 -> 131.0 mm, vias 1 -> 5
- net col3: track 111.7 -> 156.1 mm, vias 1 -> 9
- net col2: track 134.4 -> 170.1 mm, vias 1 -> 5
- net row0: track 124.2 -> 155.8 mm
- net Net-(LED10-DIN): track 58.9 -> 81.7 mm, vias 2 -> 6
- net Net-(LED14-DOUT): track 84.1 -> 104.6 mm
- net Net-(LED10-DOUT): track 81.4 -> 101.6 mm
- net Net-(LED5-DOUT): track 70.0 -> 50.8 mm, vias 3 -> 4
- net LED: track 113.6 -> 130.0 mm, vias 3 -> 5
- net Net-(LED18-VDD): track 28.6 -> 12.5 mm, vias 1 -> 2
- net Net-(LED16-DOUT): track 36.6 -> 51.1 mm, vias 2 -> 4
- net Net-(LED4-DOUT): track 37.9 -> 50.6 mm, vias 3 -> 4
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